Commit message: hide unnecessary collision files

File: resources/robots/QUB/urdf/QUB.urdf (robot description, URDF)
Before this commit: robot QUB, 14 links, 13 joints
Links:
- link L_ankle_link: geometry visual mesh filename=../meshes/L_ankle_link.STL
- link L_calf_link: geometry visual mesh filename=../meshes/L_calf_link.STL
- link L_hip_r_link: geometry visual mesh filename=../meshes/L_hip_r_link.STL
- link L_hip_y_link: geometry visual mesh filename=../meshes/L_hip_y_link.STL
- link L_thigh_link: geometry visual mesh filename=../meshes/L_thigh_link.STL
- link R_ankle_link: geometry visual mesh filename=../meshes/R_ankle_link.STL
- link R_calf_link: geometry visual mesh filename=../meshes/R_calf_link.STL
- link R_hip_r_link: geometry visual mesh filename=../meshes/R_hip_r_link.STL
- link R_hip_y_link: geometry visual mesh filename=../meshes/R_hip_y_link.STL
- link R_thigh_link: geometry visual mesh filename=../meshes/R_thigh_link.STL
